Commit message: change simulation driver to robosense

File: src/testRange/bot_description/urdf/VLP-16.urdf.xacro (robot description, xacro)
@@ -2,5 +2,5 @@
 <robot xmlns:xacro="http://www.ros.org/wiki/xacro" name="VLP-16">
   <xacro:property name="M_PI" value="3.1415926535897931" />
-  <xacro:macro name="VLP-16" params="*origin parent:=base_link name:=velodyne topic:=/velodyne_points hz:=10 lasers:=16 samples:=1875 collision_range:=0.3 min_range:=0.3 max_range:=130.0 noise:=0.008 min_angle:=-${M_PI} max_angle:=${M_PI} gpu:=false">
+  <xacro:macro name="VLP-16" params="*origin parent:=base_link name:=velodyne topic:=/velodyne_points hz:=10 lasers:=16 samples:=1875 collision_range:=0.3 min_range:=0.9 max_range:=130.0 noise:=0.008 min_angle:=-${M_PI} max_angle:=${M_PI} gpu:=false">
     <joint name="${name}_base_mount_joint" type="fixed">
       <xacro:insert_block name="origin" />

File: src/testRange/bot_description/urdf/turtlebot3_waffle_pi.urdf.xacro (robot description, xacro)
@@ -134,8 +134,13 @@
   <link name="imu_link"/>
   <xacro:property name="gpu" value="true" />
-  <xacro:include filename="$(find bot_description)/urdf/VLP-16.urdf.xacro"/>
-  <xacro:VLP-16 parent="base_link" name="velodyne" topic="/velodyne_points" hz="10" samples="440" gpu="${gpu}">
+  <xacro:include filename="$(find robosense_description)/urdf/RS-16.urdf.xacro"/>
+  <xacro:RS-16 parent="base_link" name="robosense" topic="/rs_points" hz="20" samples="900" gpu="${gpu}">
     <origin xyz="-0.064 0 0.1" rpy="0 0 0"/>
-  </xacro:VLP-16>
+  </xacro:RS-16>
+  <!-- <xacro:property name="gpu" value="true" /> -->
+  <!-- <xacro:include filename="$(find bot_description)/urdf/VLP-16.urdf.xacro"/> -->
+  <!-- <xacro:VLP-16 parent="base_link" name="velodyne" topic="/velodyne_points" hz="10" samples="440" gpu="${gpu}"> -->
+    <!-- <origin xyz="-0.064 0 0.1" rpy="0 0 0"/> -->
+  <!-- </xacro:VLP-16> -->
   <!-- <xacro:include filename="$(find velodyne_description)/urdf/HDL-32E.urdf.xacro"/> -->
   <!-- <xacro:HDL-32E parent="base_link" name="velodyne2" topic="/velodyne_points2" hz="10" samples="220" gpu="${gpu}"> -->
