Commit message: add 2d surpport

File: src/testRange/bot_description/urdf/turtlebot3_waffle_pi.urdf.xacro (robot description, xacro)
@@ -133,5 +133,5 @@
   </joint>
   <link name="imu_link"/>
-  <xacro:property name="gpu" value="false" />
+  <xacro:property name="gpu" value="true" />
   <xacro:include filename="$(find robosense_description)/urdf/RS-16.urdf.xacro"/>
   <xacro:RS-16 parent="base_link" name="robosense" topic="/rs_points" hz="20" samples="900" gpu="${gpu}">
